Commit message: 33012

File: luckrobot_ws/install/robot_display/share/robot_display/urdf/0robot.SLDASM.urdf (robot description, URDF)
Before this commit: robot robot_display, 7 links, 6 joints
Links:
- removed link livox_link
- added link livox_frame, mass 0.052593; collision mesh filename=package://robot_display/meshes/livox_link.STL; visual mesh filename=package://robot_display/meshes/livox_link.STL
Joints:
- joint livox_joint: child livox_link -> livox_frame
- joint screw_joint: limit lower=0 upper=0 effort=0 velocity=0 -> lower=-0.2 upper=0 effort=100 velocity=0.1; origin xyz=0.061648 5E-05 0.48875 rpy=0 0 0 -> xyz=0.061648 5E-05 0.671 rpy=0 0 0

Commit message: 2026472002

File: luckrobot_ws/install/robot_display/share/robot_display/urdf/0robot.SLDASM.urdf (robot description, URDF)
Before this commit: robot robot_display, 7 links, 6 joints
Links:
- added link camera_poo_link, mass 0.0326390241085313; collision mesh filename=package://robot_display/meshes/camera_link.STL; visual mesh filename=package://robot_display/meshes/camera_link.STL
- link camera_link: mass 0.032639 -> None; geometry 
- link livox_frame: mass 0.052593 -> 0.0525930263369941
- link screw_link: mass 0.266367645981795 -> 0.477619946924312
- link wheel_right_link: mass 0.31548 -> 0.315479735504946
Joints:
- added joint camera_poo_to_camera_joint: type fixed, parent camera_poo_link, child camera_link, origin xyz=0.02292 0 0 rpy=0 0 0
- joint camera_joint: axis 0 0 0 -> (none); child camera_link -> camera_poo_link; origin xyz=0.067499 6.1597E-05 0.78446 rpy=0 0 0 -> xyz=0.0336516678874285 0.0474500000000005 0.324490381056767 rpy=0 0.5235987755983 0; parent base_link -> screw_link
- joint livox_joint: axis 0 0 0 -> (none); origin xyz=0.017002 5.3506E-05 0.87097 rpy=0 0.34907 0.00016022 -> xyz=0.0170020182229269 5.3506078218414E-05 0.87097369906952 rpy=0 0.349065850398866 0.000160221167896802
- joint screw_joint: origin xyz=0.061648 5E-05 0.671 rpy=0 0 0 -> xyz=0.0616483321125747 5.00000000000496E-05 0.671 rpy=0 0 0

Commit message: 2026482132

File: luckrobot_ws/install/robot_display/share/robot_display/urdf/0robot.SLDASM.urdf (robot description, URDF)
Before this commit: robot robot_display, 8 links, 7 joints
Links:
- added link camera_init
- added link livox_body
- added link livox_poo_link, mass 0.0525930263369941; collision mesh filename=package://robot_display/meshes/livox_link.STL; visual mesh filename=package://robot_display/meshes/livox_link.STL
- link livox_frame: mass 0.0525930263369941 -> None; geometry 
Joints:
- added joint livox_frame_to_body_joint: type fixed, parent livox_frame, child livox_body, origin xyz=0.001 0.02329 -0.04412 rpy=0 0 0
- added joint livox_frame_to_camera_init_joint: type fixed, parent livox_frame, child camera_init, origin xyz=0 0 0 rpy=0 0 0
- added joint livox_poo_to_livox_joint: type fixed, parent livox_poo_link, child livox_frame, origin xyz=0 0 0.02108 rpy=0 0 0
- joint livox_joint: child livox_frame -> livox_poo_link

Commit message: 20264101053

File: luckrobot_ws/install/robot_display/share/robot_display/urdf/0robot.SLDASM.urdf (robot description, URDF)
Before this commit: robot robot_display, 11 links, 10 joints
Links:
- removed link camera_init
- removed link livox_body
- added link body
Joints:
- removed joint livox_frame_to_body_joint
- removed joint livox_frame_to_camera_init_joint
- added joint body_to_base_footprint_joint: type fixed, parent body, child base_footprint, origin xyz=0.274505096 -0.023340782 -0.811089435 rpy=0.0000583155 -0.3490658504 -0.000170503

Commit message: Localization完成3D点云匹配定位

File: luckrobot_ws/install/robot_display/share/robot_display/urdf/0robot.SLDASM.urdf (robot description, URDF)
Before this commit: robot robot_display, 10 links, 9 joints
Joints:
- joint body_to_base_footprint_joint: origin xyz=0.274505096 -0.023340782 -0.811089435 rpy=0.0000583155 -0.3490658504 -0.000170503 -> xyz=-0.0194585 -0.0233408 -0.8560610 rpy=0 0 0

File: luckrobot_ws/src/robot_display/urdf/0robot.SLDASM.urdf (robot description, URDF)
Before this commit: robot robot_display, 10 links, 9 joints
Joints:
- joint body_to_base_footprint_joint: origin xyz=0.274505096 -0.023340782 -0.811089435 rpy=0.0000583155 -0.3490658504 -0.000170503 -> xyz=-0.0194585 -0.0233408 -0.8560610 rpy=0 0 0

Commit message: 20264111743

File: luckrobot_ws/install/robot_display/share/robot_display/urdf/0robot.SLDASM.urdf (robot description, URDF)
Before this commit: robot robot_display, 10 links, 9 joints
Links:
- added link imu_link
Joints:
- added joint livox_frame_to_livox_body_joint: type fixed, parent livox_frame, child imu_link, origin xyz=0.011 0.02329 -0.04412 rpy=0 0 0

File: luckrobot_ws/src/robot_display/urdf/0robot.SLDASM.urdf (robot description, URDF)
Before this commit: robot robot_display, 10 links, 9 joints
Links:
- added link imu_link
Joints:
- added joint livox_frame_to_livox_body_joint: type fixed, parent livox_frame, child imu_link, origin xyz=0.011 0.02329 -0.04412 rpy=0 0 0

Commit message: 20264131119

File: luckrobot_ws/install/robot_display/share/robot_display/urdf/0robot.SLDASM.urdf (robot description, URDF)
Before this commit: robot robot_display, 11 links, 10 joints
Links:
- removed link camera_link
- removed link camera_poo_link
- link screw_link: mass 0.477619946924312 -> 0.510258972883763
Joints:
- removed joint camera_joint
- removed joint camera_poo_to_camera_joint
- joint body_to_base_footprint_joint: origin xyz=-0.0194585 -0.0233408 -0.8560610 rpy=0 0 0 -> xyz=-0.0139987 -0.0233413 -0.8458771 rpy=0 0 0
- joint livox_joint: origin xyz=0.0170020182229269 5.3506078218414E-05 0.87097369906952 rpy=0 0.349065850398866 0.000160221167896802 -> xyz=0.00299873713924339 5.12624561495789E-05 0.858417099999998 rpy=0 0 0
